Commit message: Latest update

File: urdf/schoolbus.urdf (robot description, URDF)
Before this commit: robot schoolbus, 12 links, 11 joints
Links:
- added link base_footprint
Joints:
- added joint base_footprint: type fixed, parent base_footprint, child base_link, origin xyz=0 0 0 rpy=0 0 0, axis 0 0 0

Commit message: New URDF

File: urdf/schoolbus.urdf (robot description, URDF)
Before this commit: robot schoolbus, 13 links, 12 joints
Links:
- link 3d_lidar_link: mass 0.57482 -> 0.5715
Joints:
- joint 3d_lidar: origin xyz=0.1778 0 0.9383 rpy=0 0 0 -> xyz=0.1778 0 0.94942 rpy=0 0 0
- joint imu: origin xyz=0 0 0.6992 rpy=0 0 0 -> xyz=0.1778 0 0.86122 rpy=0 0 0
